File: _saved_sk6812-demo.sch (KiCad schematic (older format))
At the start: 11 parts, among them U1 Photon

Commit message: Fixing power nets
Parts:
- R1, R2: footprint (none) -> Resistors_SMD:R_0805
Changed lines of the file:
@@
 $EndComp
 $Comp
-L GND #PWR18
+L GND #PWR01
 U 1 1 583D0AA9
 P 2400 6150
-F 0 "#PWR18" H 2400 5900 50  0001 C CNN
+F 0 "#PWR01" H 2400 5900 50  0001 C CNN
 F 1 "GND" H 2400 6000 50  0000 C CNN
 F 2 "" H 2400 6150 50  0000 C CNN
@@
 $EndComp
 $Comp
-L GND #PWR8
+L GND #PWR02
 U 1 1 583D0E0A
 P 8750 2750
-F 0 "#PWR8" H 8750 2500 50  0001 C CNN
+F 0 "#PWR02" H 8750 2500 50  0001 C CNN
 F 1 "GND" H 8750 2600 50  0000 C CNN
 F 2 "" H 8750 2750 50  0000 C CNN
@@
 $EndComp
 $Comp
-L GND #PWR7
+L GND #PWR03
 U 1 1 583D0E4F
 P 7150 2750
-F 0 "#PWR7" H 7150 2500 50  0001 C CNN
+F 0 "#PWR03" H 7150 2500 50  0001 C CNN
 F 1 "GND" H 7150 2600 50  0000 C CNN
 F 2 "" H 7150 2750 50  0000 C CNN
@@
 $EndComp
 $Comp
-L GND #PWR6
+L GND #PWR04
 U 1 1 583D0EF9
 P 5600 2750
-F 0 "#PWR6" H 5600 2500 50  0001 C CNN
+F 0 "#PWR04" H 5600 2500 50  0001 C CNN
 F 1 "GND" H 5600 2600 50  0000 C CNN
 F 2 "" H 5600 2750 50  0000 C CNN
@@
 $EndComp
 $Comp
-L GND #PWR5
+L GND #PWR05
 U 1 1 583D0F37
 P 4050 2750
-F 0 "#PWR5" H 4050 2500 50  0001 C CNN
+F 0 "#PWR05" H 4050 2500 50  0001 C CNN
 F 1 "GND" H 4050 2600 50  0000 C CNN
 F 2 "" H 4050 2750 50  0000 C CNN
@@
 $EndComp
 $Comp
-L +5V #PWR13
+L +5V #PWR06
 U 1 1 583D1010
 P 2250 3900
-F 0 "#PWR13" H 2250 3750 50  0001 C CNN
+F 0 "#PWR06" H 2250 3750 50  0001 C CNN
 F 1 "+5V" H 2250 4040 50  0000 C CNN
 F 2 "" H 2250 3900 50  0000 C CNN
@@
 $EndComp
 $Comp
-L +5V #PWR1
+L +5V #PWR07
 U 1 1 583D10FF
 P 5200 2000
-F 0 "#PWR1" H 5200 1850 50  0001 C CNN
+F 0 "#PWR07" H 5200 1850 50  0001 C CNN
 F 1 "+5V" H 5200 2140 50  0000 C CNN
 F 2 "" H 5200 2000 50  0000 C CNN
@@
 $EndComp
 $Comp
-L +5V #PWR2
+L +5V #PWR08
 U 1 1 583D113D
 P 6750 2000
-F 0 "#PWR2" H 6750 1850 50  0001 C CNN
+F 0 "#PWR08" H 6750 1850 50  0001 C CNN
 F 1 "+5V" H 6750 2140 50  0000 C CNN
 F 2 "" H 6750 2000 50  0000 C CNN
@@
 $EndComp
 $Comp
-L +5V #PWR3
+L +5V #PWR09
 U 1 1 583D1258
 P 8300 2000
-F 0 "#PWR3" H 8300 1850 50  0001 C CNN
+F 0 "#PWR09" H 8300 1850 50  0001 C CNN
 F 1 "+5V" H 8300 2140 50  0000 C CNN
 F 2 "" H 8300 2000 50  0000 C CNN
@@
 $EndComp
 $Comp
-L +5V #PWR4
+L +5V #PWR010
 U 1 1 583D1296
 P 9900 2000
-F 0 "#PWR4" H 9900 1850 50  0001 C CNN
+F 0 "#PWR010" H 9900 1850 50  0001 C CNN
 F 1 "+5V" H 9900 2140 50  0000 C CNN
 F 2 "" H 9900 2000 50  0000 C CNN
@@
 NEO_3
 $Comp
-L GND #PWR17
+L GND #PWR011
 U 1 1 583D2F21
 P 8750 4250
-F 0 "#PWR17" H 8750 4000 50  0001 C CNN
+F 0 "#PWR011" H 8750 4000 50  0001 C CNN
 F 1 "GND" H 8750 4100 50  0000 C CNN
 F 2 "" H 8750 4250 50  0000 C CNN
@@
 $EndComp
 $Comp
-L GND #PWR16
+L GND #PWR012
 U 1 1 583D2F27
 P 7150 4250
-F 0 "#PWR16" H 7150 4000 50  0001 C CNN
+F 0 "#PWR012" H 7150 4000 50  0001 C CNN
 F 1 "GND" H 7150 4100 50  0000 C CNN
 F 2 "" H 7150 4250 50  0000 C CNN
@@
 $EndComp
 $Comp
-L GND #PWR15
+L GND #PWR013
 U 1 1 583D2F2D
 P 5600 4250
-F 0 "#PWR15" H 5600 4000 50  0001 C CNN
+F 0 "#PWR013" H 5600 4000 50  0001 C CNN
 F 1 "GND" H 5600 4100 50  0000 C CNN
 F 2 "" H 5600 4250 50  0000 C CNN
@@
 $EndComp
 $Comp
-L GND #PWR14
+L GND #PWR014
 U 1 1 583D2F33
 P 4050 4250
-F 0 "#PWR14" H 4050 4000 50  0001 C CNN
+F 0 "#PWR014" H 4050 4000 50  0001 C CNN
 F 1 "GND" H 4050 4100 50  0000 C CNN
 F 2 "" H 4050 4250 50  0000 C CNN
@@
 $EndComp
 $Comp
-L +5V #PWR9
+L +5V #PWR015
 U 1 1 583D2F39
 P 5200 3500
-F 0 "#PWR9" H 5200 3350 50  0001 C CNN
+F 0 "#PWR015" H 5200 3350 50  0001 C CNN
 F 1 "+5V" H 5200 3640 50  0000 C CNN
 F 2 "" H 5200 3500 50  0000 C CNN
@@
 $EndComp
 $Comp
-L +5V #PWR10
+L +5V #PWR016
 U 1 1 583D2F3F
 P 6750 3500
-F 0 "#PWR10" H 6750 3350 50  0001 C CNN
+F 0 "#PWR016" H 6750 3350 50  0001 C CNN
 F 1 "+5V" H 6750 3640 50  0000 C CNN
 F 2 "" H 6750 3500 50  0000 C CNN
@@
 $EndComp
 $Comp
-L +5V #PWR11
+L +5V #PWR017
 U 1 1 583D2F45
 P 8300 3500
-F 0 "#PWR11" H 8300 3350 50  0001 C CNN
+F 0 "#PWR017" H 8300 3350 50  0001 C CNN
 F 1 "+5V" H 8300 3640 50  0000 C CNN
 F 2 "" H 8300 3500 50  0000 C CNN
@@
 $EndComp
 $Comp
-L +5V #PWR12
+L +5V #PWR018
 U 1 1 583D2F4B
 P 9900 3500
-F 0 "#PWR12" H 9900 3350 50  0001 C CNN
+F 0 "#PWR018" H 9900 3350 50  0001 C CNN
 F 1 "+5V" H 9900 3640 50  0000 C CNN
 F 2 "" H 9900 3500 50  0000 C CNN
@@
 NEO_7
 $Comp
-L PWR_FLAG #FLG1
+L PWR_FLAG #FLG019
 U 1 1 583D3561
 P 2050 4000
-F 0 "#FLG1" H 2050 4095 50  0001 C CNN
+F 0 "#FLG019" H 2050 4095 50  0001 C CNN
 F 1 "PWR_FLAG" H 2050 4180 50  0000 C CNN
 F 2 "" H 2050 4000 50  0000 C CNN
@@
 $EndComp
 $Comp
-L PWR_FLAG #FLG2
+L PWR_FLAG #FLG020
 U 1 1 583D35A6
 P 2150 6000
-F 0 "#FLG2" H 2150 6095 50  0001 C CNN
+F 0 "#FLG020" H 2150 6095 50  0001 C CNN
 F 1 "PWR_FLAG" H 2150 6180 50  0000 C CNN
 F 2 "" H 2150 6000 50  0000 C CNN
@@
 F 0 "R1" V 3580 3300 50  0000 C CNN
 F 1 "R" V 3500 3300 50  0000 C CNN
-F 2 "" V 3430 3300 50  0000 C CNN
+F 2 "Resistors_SMD:R_0805" V 3430 3300 50  0001 C CNN
 F 3 "" H 3500 3300 50  0000 C CNN
 	1    3500 3300
@@
 F 0 "R2" V 3730 4400 50  0000 C CNN
 F 1 "R" V 3650 4400 50  0000 C CNN
-F 2 "" V 3580 4400 50  0000 C CNN
+F 2 "Resistors_SMD:R_0805" V 3580 4400 50  0001 C CNN
 F 3 "" H 3650 4400 50  0000 C CNN
 	1    3650 4400
